File: IoTBoard.kicad_pcb (KiCad board)
At the start: 2 copper layers, 84.8 x 84.8 mm, 56 parts, among them J1 DHT22, J2 OLED, J3 LED_Conn, Q1 AO3401A, SW1 SW_Push, SW2 SW_Push

Commit message: Changed PCB
Fixed errors
Parts:
- C10, C11, C12, C13, C14, C15, C16, C17, C19, C20, C6, C7, C8, C9: value C -> 100nF
- C4, C5: value C -> 10nF
- D9: footprint LED_SMD:LED_Avago_PLCC6_3x2.8mm -> LED_SMD:LED_WS2812_PLCC6_5.0x5.0mm_P1.6mm
- R1, R3, R7: value R -> 10K
- R8: value R -> 100K
- SW1, SW2: footprint Button_Switch_SMD:SW_Push_1P1T_NO_6x6mm_H9.5mm -> Button_Switch_SMD:SW_SPST_Omron_B3FS-105xP
- moved R6 9.53 mm to (118.6, 88.6)
- moved R5 9.46 mm to (120.8, 88.6)
- moved R4 9.39 mm to (123.0, 88.6)
- moved D9 8.25 mm to (120.8, 94.4)
Connections:
- J1 pad 2: unconnected-(J1-Pin_2-Pad2) -> DHT22_DATA
- J1 pad 3: DHT22_DATA -> unconnected-(J1-Pin_3-Pad3)
Routing:
- net LED_B: track 28.5 -> 19.7 mm
- net LED_G: track 24.6 -> 15.9 mm
- net LED_R: track 18.4 -> 12.0 mm
Other:
- board text added: "IoT EduBoard"
- board text added: "Project: IoT Education Board v.5 Author: Michal Kubascik Department of Technical Cybernetics Faculty of Management Science and Informatics"
- board text removed: "IoT Board v.1"
- board text removed: "Project: IoT Board - Summer school v.4 Author: Michal Kubascik Department of Technical Cybernetics Faculty of Management Science and Informatics"
