File: IoTBoard.kicad_sch (KiCad schematic)
At the start: 56 parts, among them J1 DHT22, J2 OLED, J3 LED_Conn, Q1 AO3401A, SW1 SW_Push, SW2 SW_Push

Commit message: Changed PCB
Fixed errors
Parts:
- C10, C11, C12, C13, C14, C15, C16, C17, C19, C20, C6, C7, C8, C9: value C -> 100nF
- C4, C5: value C -> 10nF
- D9: footprint LED_SMD:LED_Avago_PLCC6_3x2.8mm -> LED_SMD:LED_WS2812_PLCC6_5.0x5.0mm_P1.6mm
- R1, R3, R7: value R -> 10K
- R8: value R -> 100K
- SW1, SW2: footprint Button_Switch_SMD:SW_Push_1P1T_NO_6x6mm_H9.5mm -> Button_Switch_SMD:SW_SPST_Omron_B3FS-105xP
Connections:
- net DHT22_DATA: now also J1.2 (Pin_2); no longer J1.3 (Pin_3)
